Commit message: Add USD file and fix bugs.

File: model/kurokun.urdf (robot description, URDF)
Before this commit: robot kurokun, 15 links, 14 joints
Links:
- added link head_link, mass 0.250; collision box size=0.065 0.07528 0.042; visual box size=0.065 0.07528 0.042
- link base_link: mass 0.250 -> 0.001; geometry collision box size=0.120 0.100 0.060
Joints:
- added joint head_joint: type fixed, parent base_link, child head_link, origin xyz=0.010 0 -0.045 rpy=0 0 0

Commit message: Change USD file.

File: model/kurokun.urdf (robot description, URDF)
Before this commit: robot kurokun, 16 links, 15 joints
Links:
- link left_ankle_link: geometry collision box size=0.0363 0.02472 0.04522; visual box size=0.0363 0.02472 0.04522
- link left_hip_pitch_link: geometry collision box size=0.0363 0.02472 0.04522; visual box size=0.0363 0.02472 0.04522
- link left_hip_roll_link: geometry collision box size=0.02472 0.0363 0.04522; visual box size=0.02472 0.0363 0.04522
- link left_knee_link: geometry collision box size=0.0363 0.02472 0.04522; visual box size=0.0363 0.02472 0.04522
- link right_ankle_link: geometry collision box size=0.0363 0.02472 0.04522; visual box size=0.0363 0.02472 0.04522
- link right_hip_pitch_link: geometry collision box size=0.0363 0.02472 0.04522; visual box size=0.0363 0.02472 0.04522
- link right_hip_roll_link: geometry collision box size=0.02472 0.0363 0.04522; visual box size=0.02472 0.0363 0.04522
- link right_knee_link: geometry collision box size=0.0363 0.02472 0.04522; visual box size=0.0363 0.02472 0.04522
Joints:
- joint left_ankle_to_foot: origin xyz=0 0 -0.0363 rpy=0 0 0 -> xyz=0 0 -0.03511 rpy=0 0 0
- joint left_shank_joint: origin xyz=0 0 -0.0363 rpy=0 0 0 -> xyz=0 0 -0.03511 rpy=0 0 0
- joint left_thigh_joint: origin xyz=0 0 -0.0363 rpy=0 0 0 -> xyz=0 0 -0.03511 rpy=0 0 0
- joint right_ankle_to_foot: origin xyz=0 0 -0.0363 rpy=0 0 0 -> xyz=0 0 -0.03511 rpy=0 0 0
- joint right_shank_joint: origin xyz=0 0 -0.0363 rpy=0 0 0 -> xyz=0 0 -0.03511 rpy=0 0 0
- joint right_thigh_joint: origin xyz=0 0 -0.0363 rpy=0 0 0 -> xyz=0 0 -0.03511 rpy=0 0 0

Commit message: Add deploy part.

File: model/kurokun.urdf (robot description, URDF)
Before this commit: robot kurokun, 16 links, 15 joints
Links:
- link left_shank_link: geometry collision box size=0.037 0.025 0.015; visual box size=0.037 0.025 0.015
- link left_thigh_link: geometry collision box size=0.037 0.025 0.015; visual box size=0.037 0.025 0.015
- link right_shank_link: geometry collision box size=0.037 0.025 0.015; visual box size=0.037 0.025 0.015
- link right_thigh_link: geometry collision box size=0.037 0.025 0.015; visual box size=0.037 0.025 0.015
Joints:
- joint left_ankle: origin xyz=0 0 -0.035 rpy=0 0 0 -> xyz=0 0 -0.040 rpy=0 0 0
- joint left_ankle_to_foot: origin xyz=0 0 -0.03511 rpy=0 0 0 -> xyz=0 0 -0.01011 rpy=0 0 0
- joint left_hip_pitch: origin xyz=0.03497 0.01025 0 rpy=0 0 0 -> xyz=0.03497 0.01025 -0.025 rpy=0 0 0
- joint left_knee: origin xyz=0 0 -0.035 rpy=0 0 0 -> xyz=0 0 -0.040 rpy=0 0 0
- joint left_shank_joint: origin xyz=0 0 -0.03511 rpy=0 0 0 -> xyz=0 0 -0.01011 rpy=0 0 0
- joint left_thigh_joint: origin xyz=0 0 -0.03511 rpy=0 0 0 -> xyz=0 0 -0.01011 rpy=0 0 0
- joint right_ankle: origin xyz=0 0 -0.035 rpy=0 0 0 -> xyz=0 0 -0.040 rpy=0 0 0
- joint right_ankle_to_foot: origin xyz=0 0 -0.03511 rpy=0 0 0 -> xyz=0 0 -0.01011 rpy=0 0 0
- joint right_hip_pitch: origin xyz=0.03497 -0.01025 0 rpy=0 0 0 -> xyz=0.03497 -0.01025 -0.025 rpy=0 0 0
- joint right_knee: origin xyz=0 0 -0.035 rpy=0 0 0 -> xyz=0 0 -0.040 rpy=0 0 0
- joint right_shank_joint: origin xyz=0 0 -0.03511 rpy=0 0 0 -> xyz=0 0 -0.01011 rpy=0 0 0
- joint right_thigh_joint: origin xyz=0 0 -0.03511 rpy=0 0 0 -> xyz=0 0 -0.01011 rpy=0 0 0
